File: circuit_design/circuit_design.kicad_sch (KiCad schematic)
At the start: 1 part

Commit message: pr4
Parts:
- removed R1: ~, My_Library:Resistor, symbol My_Library:Resistor
- added DD1: ~, Pr4:К155ЛА3, symbol Pr4:К155ЛА3
Connections:
- new net Vcc: DD1.14 (Vcc)
Changed lines of the file:
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@@
 	(generator_version "8.0")
 	(paper "A4")
-	(wire
-		(pts
-			(xy 90.17 64.77) (xy 90.17 74.93)
-		)
-		(stroke
-			(width 0)
-			(type default)
-		)
-	)
-	(wire
-		(pts
-			(xy 90.17 74.93) (xy 86.36 74.93)
-		)
-		(stroke
-			(width 0)
-			(type default)
-		)
-	)
-	(wire
-		(pts
-			(xy 86.36 64.77) (xy 90.17 64.77)
-		)
-		(stroke
-			(width 0)
-			(type default)
-		)
-	)
 	(symbol
-		(lib_id "My_Library:Resistor")
-		(at 86.36 69.85 0)
+		(lib_id "Pr4:К155ЛА3")
+		(at 68.58 71.12 0)
 		(unit 1)
 		(exclude_from_sim no)
@@
 		(on_board yes)
 		(dnp no)
-		(property "Reference" "R1"
-			(at 85.09 69.85 0)
+		(fields_autoplaced yes)
+		(property "Reference" "DD1"
+			(at 68.69 62.23 0)
 			(effects
 				(font
 					(size 1.27 1.27)
 				)
-				(justify left)
 			)
 		)
 		(property "Value" "~"
-			(at 88.9 71.12 0)
+			(at 68.69 64.77 0)
 			(effects
 				(font
 					(size 1.27 1.27)
 				)
-				(justify left)
 			)
 		)
-		(property "Footprint" "My_Library:Resistor"
-			(at 82.55 61.976 0)
+		(property "Footprint" "Pr4:К155ЛА3"
+			(at 68.58 78.74 0)
 			(effects
 				(font
@@
 		)
 		(property "Datasheet" ""
-			(at 86.36 69.85 0)
+			(at 68.58 66.04 0)
 			(effects
 				(font
@@
 		)
 		(property "Description" ""
-			(at 86.36 69.85 0)
+			(at 68.58 66.04 0)
 			(effects
 				(font
@@
 			)
 		)
+		(pin "14"
+		)
+		(pin "1"
+		)
 		(pin "2"
 		)
-		(pin "1"
+		(pin "3"
+		)
+		(pin "7"
 		)
 		(instances
 			(project ""
 				(path "/936cfab9-3290-4713-92ea-50f992466908"
-					(reference "R1")
+					(reference "DD1")
 					(unit 1)
 				)

Commit message: pr5
Parts:
- added unit 3 of DD1
- added unit 2 of DD1
- added unit 4 of DD1
Connections:
- removed net Vcc: DD1.14 (Vcc)

Commit message: maybe 10?
Parts:
- removed DD1: ~, Pr4:К155ЛА3, symbol Pr4:К155ЛА3
- added C1, C2: 10nF, Pr2:CAP_CERAM_L5.0D0.8, symbol Pr2:Cap К10-17Б
- added R1: 10K, Pr2:RES_CONST_L6.0D0.8, symbol Pr2:Res MF 0.125
- added R2: 2K, Pr2:RES_CONST_L6.0D0.8, symbol Pr2:Res MF 0.125
- added VT1: 2N3904, Package_TO_SOT_THT:TO-92_Inline, symbol Transistor_BJT:2N3904
- added XP1, XP2, XP3: ~, Pr7:PLS-2, symbol pr7:PLS-2
Connections:
- new net: C1.2, VT1.2 (B)
- new net: C1.1, XP1.1
- new net GND: VT1.1 (E), XP2.2, XP3.2
